File: Splinch xiao/Splinch xiao/Splinch xiao.kicad_pcb (KiCad board)
At the start: 2 copper layers, 135.8 x 106.8 mm, 68 parts, among them SW1 Switch, U2 Seeeduino Xiao nRF52840

Commit message: outline and left schem
Parts:
- added D31: Diode, ScottoKeebs_Components:Diode_SOD-123, F.Cu at (-34.8, 164.4)
- added D32: Diode, ScottoKeebs_Components:Diode_SOD-123, F.Cu at (-34.8, 167.7)
- added D33: Diode, ScottoKeebs_Components:Diode_SOD-123, F.Cu at (-34.8, 171.1)
- added D34: Diode, ScottoKeebs_Components:Diode_SOD-123, F.Cu at (-34.8, 174.4)
- added D35: Diode, ScottoKeebs_Components:Diode_SOD-123, F.Cu at (-34.8, 177.8)
- added D35'2: Diode, ScottoKeebs_Components:Diode_SOD-123, F.Cu at (-17.6, 177.8)
- added D36: Diode, ScottoKeebs_Components:Diode_SOD-123, F.Cu at (-34.8, 181.1)
- added D37: Diode, ScottoKeebs_Components:Diode_SOD-123, F.Cu at (-34.8, 184.5)
- added D38: Diode, ScottoKeebs_Components:Diode_SOD-123, F.Cu at (-29.1, 161.0)
- added D39: Diode, ScottoKeebs_Components:Diode_SOD-123, F.Cu at (-29.1, 164.4)
- added D40: Diode, ScottoKeebs_Components:Diode_SOD-123, F.Cu at (-29.1, 167.7)
- added D41: Diode, ScottoKeebs_Components:Diode_SOD-123, F.Cu at (-29.1, 171.1)
- added D42: Diode, ScottoKeebs_Components:Diode_SOD-123, F.Cu at (-29.1, 174.4)
- added D43: Diode, ScottoKeebs_Components:Diode_SOD-123, F.Cu at (-29.1, 177.8)
- added D44: Diode, ScottoKeebs_Components:Diode_SOD-123, F.Cu at (-29.1, 181.1)
- added D45: Diode, ScottoKeebs_Components:Diode_SOD-123, F.Cu at (-29.1, 184.5)
- added D46: Diode, ScottoKeebs_Components:Diode_SOD-123, F.Cu at (-23.3, 161.0)
- added D47: Diode, ScottoKeebs_Components:Diode_SOD-123, F.Cu at (-23.3, 164.4)
- added D48: Diode, ScottoKeebs_Components:Diode_SOD-123, F.Cu at (-23.3, 167.7)
- added D49: Diode, ScottoKeebs_Components:Diode_SOD-123, F.Cu at (-23.3, 171.1)
- added D50: Diode, ScottoKeebs_Components:Diode_SOD-123, F.Cu at (-23.3, 174.4)
- added D51: Diode, ScottoKeebs_Components:Diode_SOD-123, F.Cu at (-23.3, 177.8)
- added D52: Diode, ScottoKeebs_Components:Diode_SOD-123, F.Cu at (-23.3, 181.1)
- added D53: Diode, ScottoKeebs_Components:Diode_SOD-123, F.Cu at (-23.3, 184.5)
- added D54: Diode, ScottoKeebs_Components:Diode_SOD-123, F.Cu at (-17.6, 161.0)
- added D55: Diode, ScottoKeebs_Components:Diode_SOD-123, F.Cu at (-17.6, 164.4)
- added D56: Diode, ScottoKeebs_Components:Diode_SOD-123, F.Cu at (-17.6, 167.7)
- added D57: Diode, ScottoKeebs_Components:Diode_SOD-123, F.Cu at (-17.6, 171.1)
- added D58: Diode, ScottoKeebs_Components:Diode_SOD-123, F.Cu at (-17.6, 174.4)
- added D6: Diode, ScottoKeebs_Components:Diode_SOD-123, F.Cu at (-34.8, 161.0)
- added R3: 806k, Resistor_SMD:R_0805_2012Metric_Pad1.20x1.40mm_HandSolder, F.Cu at (15.1, 167.4)
- added R4: 2m, Resistor_SMD:R_0805_2012Metric_Pad1.20x1.40mm_HandSolder, F.Cu at (15.1, 170.4)
- added S30: Keyswitch, keyswitches.pretty-master:Kailh_socket_PG1350, F.Cu at (-27.6, 73.2)
- added S31: Keyswitch, keyswitches.pretty-master:Kailh_socket_PG1350, F.Cu at (-27.6, 92.4)
- added S32: Keyswitch, keyswitches.pretty-master:Kailh_socket_PG1350, F.Cu at (-27.6, 111.5)
- added S33: Keyswitch, keyswitches.pretty-master:Kailh_socket_PG1350, F.Cu at (-27.6, 130.7)
- added S33'2: Keyswitch, keyswitches.pretty-master:Kailh_socket_PG1350, F.Cu at (70.8, 149.8)
- added S34: Keyswitch, keyswitches.pretty-master:Kailh_socket_PG1350, F.Cu at (-27.6, 149.8)
- added S35: Keyswitch, keyswitches.pretty-master:Kailh_socket_PG1350, F.Cu at (-7.93, 73.2)
- added S36: Keyswitch, keyswitches.pretty-master:Kailh_socket_PG1350, F.Cu at (-7.93, 92.4)
- added S37: Keyswitch, keyswitches.pretty-master:Kailh_socket_PG1350, F.Cu at (-7.93, 111.5)
- added S38: Keyswitch, keyswitches.pretty-master:Kailh_socket_PG1350, F.Cu at (-7.93, 130.7)
- added S39: Keyswitch, keyswitches.pretty-master:Kailh_socket_PG1350, F.Cu at (-7.93, 149.8)
- added S40: Keyswitch, keyswitches.pretty-master:Kailh_socket_PG1350, F.Cu at (11.7, 73.2)
- added S41: Keyswitch, keyswitches.pretty-master:Kailh_socket_PG1350, F.Cu at (11.7, 92.4)
- added S42: Keyswitch, keyswitches.pretty-master:Kailh_socket_PG1350, F.Cu at (11.7, 111.5)
- added S43: Keyswitch, keyswitches.pretty-master:Kailh_socket_PG1350, F.Cu at (11.7, 130.7)
- added S44: Keyswitch, keyswitches.pretty-master:Kailh_socket_PG1350, F.Cu at (11.7, 149.8)
- added S45: Keyswitch, keyswitches.pretty-master:Kailh_socket_PG1350, F.Cu at (31.4, 73.2)
- added S46: Keyswitch, keyswitches.pretty-master:Kailh_socket_PG1350, F.Cu at (31.4, 92.4)
- added S47: Keyswitch, keyswitches.pretty-master:Kailh_socket_PG1350, F.Cu at (31.4, 111.5)
- added S48: Keyswitch, keyswitches.pretty-master:Kailh_socket_PG1350, F.Cu at (31.4, 130.7)
- added S49: Keyswitch, keyswitches.pretty-master:Kailh_socket_PG1350, F.Cu at (31.4, 149.8)
- added S50: Keyswitch, keyswitches.pretty-master:Kailh_socket_PG1350, F.Cu at (51.1, 73.2)
- added S51: Keyswitch, keyswitches.pretty-master:Kailh_socket_PG1350, F.Cu at (51.1, 92.4)
- added S52: Keyswitch, keyswitches.pretty-master:Kailh_socket_PG1350, F.Cu at (51.1, 111.5)
- added S53: Keyswitch, keyswitches.pretty-master:Kailh_socket_PG1350, F.Cu at (51.1, 130.7)
- added S54: Keyswitch, keyswitches.pretty-master:Kailh_socket_PG1350, F.Cu at (51.1, 149.8)
- added S55: Keyswitch, keyswitches.pretty-master:Kailh_socket_PG1350, F.Cu at (70.8, 73.2)
- added S56: Keyswitch, keyswitches.pretty-master:Kailh_socket_PG1350, F.Cu at (70.8, 92.4)
- added S57: Keyswitch, keyswitches.pretty-master:Kailh_socket_PG1350, F.Cu at (70.8, 111.5)
- added S58: Keyswitch, keyswitches.pretty-master:Kailh_socket_PG1350, F.Cu at (70.8, 130.7)
- added SW2: Switch, ScottoKeebs_Components:Switch_MSK12C02, F.Cu at (17.5, 162.8)
- added TP5: TestPoint, TestPoint:TestPoint_Pad_D3.0mm, F.Cu at (10.2, 161.9)
- added TP6: TestPoint, TestPoint:TestPoint_Pad_D3.0mm, F.Cu at (10.2, 166.9)
- added TP7: TestPoint, TestPoint:TestPoint_Pad_D3.0mm, F.Cu at (10.2, 172.0)
- added TP8: TestPoint, TestPoint:TestPoint_Pad_D3.0mm, F.Cu at (10.2, 177.0)
- added U1: Seeeduino Xiao nRF52840, marbastlib-xp-promicroish:Xiao_nRF52840_ACH, F.Cu at (-3.51, 170.6)
Other:
- board size 135.8 x 106.8 mm -> 134.1 x 104.5 mm

Commit message: did some of the other galf
Parts:
- moved S32 437.4 mm to (408.9, 138.0), turned to -15 degrees
- moved S34 420.6 mm to (389.7, 97.3)
- moved S33 420.5 mm to (389.7, 79.2)
- moved S35 399.9 mm to (389.7, 115.4)
- moved S36 398.6 mm to (388.6, 133.5)
- moved S39 383.3 mm to (371.6, 96.2)
- moved S38 383.2 mm to (371.6, 78.1)
- moved S37 383.0 mm to (371.6, 60.0)
- moved S40 362.2 mm to (371.6, 114.3)
- moved S41 361.0 mm to (370.5, 132.4)
- moved S44 346.5 mm to (353.5, 92.8)
- moved S43 346.3 mm to (353.5, 74.7)
- moved S42 346.2 mm to (353.5, 56.6)
- moved S33'2 331.1 mm to (389.7, 61.1)
- moved S45 324.3 mm to (353.5, 110.9)
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Routing:
- net row 3: track 118.9 -> 0.00 mm, vias 10 -> 0
- net row 2: track 118.5 -> 0.00 mm, vias 10 -> 0
- net row 0: track 116.3 -> 0.00 mm
- net row 1: track 96.4 -> 0.00 mm, vias 10 -> 0
- net col 3: track 78.3 -> 0.00 mm
- net col 1: track 73.1 -> 0.00 mm
- net col 2: track 73.1 -> 0.00 mm
- net col 6: track 72.4 -> 0.00 mm
- net row 4: track 61.1 -> 0.00 mm, vias 4 -> 0
- net col 5: track 54.3 -> 0.00 mm
- net col 4: track 54.3 -> 0.00 mm
- net Net-(D28-A): track 8.04 -> 0.00 mm
- net Net-(D35'1-A): track 8.04 -> 0.00 mm
- net Net-(D7-A): track 8.04 -> 0.00 mm
- net Net-(D24-A): track 8.04 -> 0.00 mm
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Other:
- board size 134.1 x 104.5 mm -> 244.9 x 104.5 mm

Commit message: case' wiring and more
Parts:
- added REF**: MouseBite-Part_2.0x2.0mm_outset_D0.5mm_P0.85mm_3h, Panelization:MouseBite-Part_2.0x2.0mm_outset_D0.5mm_P0.85mm_3h, F.Cu at (282.8, 91.6)
- added REF**: MouseBite-Part_2.0x2.0mm_outset_D0.5mm_P0.85mm_3h, Panelization:MouseBite-Part_2.0x2.0mm_outset_D0.5mm_P0.85mm_3h, F.Cu at (282.8, 57.7)
- added REF**: MouseBite-Part_2.0x2.0mm_outset_D0.5mm_P0.85mm_3h, Panelization:MouseBite-Part_2.0x2.0mm_outset_D0.5mm_P0.85mm_3h, F.Cu at (281.1, 125.6)
- added REF**: MouseBite-Part_2.0x2.0mm_outset_D0.5mm_P0.85mm_3h, Panelization:MouseBite-Part_2.0x2.0mm_outset_D0.5mm_P0.85mm_3h, F.Cu at (281.1, 91.6)
- added REF**: MouseBite-Part_2.0x2.0mm_outset_D0.5mm_P0.85mm_3h, Panelization:MouseBite-Part_2.0x2.0mm_outset_D0.5mm_P0.85mm_3h, F.Cu at (282.8, 125.6)
- added REF**: MouseBite-Part_2.0x2.0mm_outset_D0.5mm_P0.85mm_3h, Panelization:MouseBite-Part_2.0x2.0mm_outset_D0.5mm_P0.85mm_3h, F.Cu at (281.1, 57.7)
- D31, D32, D33, D34, D35, D35'2, D36, D37, D38, D39, D40, D41, D42, D43, D44, D45, D46, D47, D48, D49, D50, D51, D52, D53, D54, D55, D56, D57, D58, D6, TP5, TP6, TP7, TP8: moved to B.Cu
- R2: value 2m -> 2M
- moved D37 299.9 mm to (362.6, 57.1), turned to -90 degrees
- moved D35'2 296.6 mm to (386.9, 57.6), turned to 180 degrees
- moved U1 286.4 mm to (405.6, 64.4)
- moved D42 284.3 mm to (344.5, 53.7), turned to -90 degrees
- moved D33 279.9 mm to (380.7, 76.3), turned to -90 degrees
- moved R4 279.6 mm to (405.6, 62.2)
- moved D6 276.2 mm to (398.8, 83.1), turned to -90 degrees
- moved R3 274.9 mm to (405.6, 64.4)
- moved D43 270.6 mm to (344.5, 71.8), turned to -90 degrees
- moved D34 267.5 mm to (380.7, 94.4), turned to -90 degrees
- moved D51 267.1 mm to (308.3, 61.6), turned to -90 degrees
- moved D47 264.6 mm to (326.4, 56.0), turned to -90 degrees
- moved D31 264.5 mm to (398.8, 101.2), turned to -90 degrees
- moved D38 260.3 mm to (362.6, 75.2), turned to -90 degrees
- moved D44 257.1 mm to (344.5, 89.9), turned to -90 degrees
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Connections:
- U1 pad 11: col 0' -> row 0'
- U1 pad 12: col 1' -> row 1'
- U1 pad 13: col 2' -> row 2'
- U1 pad 14: col 3' -> row 4'
- U1 pad 17: col 6' -> row 3'
- U1 pad 18: col 5' -> col 0'
- U1 pad 2: row 0' -> col 6'
- U1 pad 22: GND -> unconnected-(U1-GND-Pad22)
- U1 pad 3: row 1' -> col 5'
- U1 pad 4: row 2' -> col 4'
- U1 pad 5: row 3' -> col 3'
- U1 pad 6: row 4' -> col 1'
- U1 pad 7: col 4' -> col 2'
- U1 pad 9: GND -> GND'
- U2 pad 11: col 0 -> col 6
- U2 pad 12: col 1 -> col 5
- U2 pad 13: col 2 -> col 4
- U2 pad 17: col 6 -> col 0
- U2 pad 18: col 5 -> col 1
- U2 pad 22: GND -> unconnected-(U2-GND-Pad22)
- U2 pad 7: col 4 -> col 2
Routing:
- net col 6: track 0.00 -> 184.1 mm
- net col 6': track 0.00 -> 176.3 mm, vias 0 -> 8
- net col 5: track 0.00 -> 173.6 mm, vias 0 -> 8
- net bat-: track 0.00 -> 162.0 mm, vias 0 -> 2
- net col 5': track 0.00 -> 161.9 mm, vias 0 -> 8
- net col 3: track 0.00 -> 156.5 mm, vias 0 -> 10
- net row 3: track 0.00 -> 156.4 mm, vias 0 -> 3
- net col 4: track 0.00 -> 152.1 mm, vias 0 -> 8
- net col 2: track 0.00 -> 149.9 mm, vias 0 -> 11
- net row 3': track 0.00 -> 149.3 mm
- net col 3': track 0.00 -> 143.7 mm, vias 0 -> 10
- net row 2': track 0.00 -> 142.6 mm
- net row 2: track 0.00 -> 140.7 mm, vias 0 -> 1
- net col 4': track 0.00 -> 140.6 mm, vias 0 -> 8
- net row 0': track 0.00 -> 136.8 mm
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- added copper zone on B.Cu, net (none)
- added copper zone on F.Cu, net (none)
Other:
- board size 244.9 x 104.5 mm -> 270.4 x 104.8 mm

Commit message: added silk screen and reade me
Parts:
- added G***: LOGO, splinch photos:potter on a broom, F.Cu at (154.4, 120.5)
- added G***: LOGO, splinch photos:potter on a broom, F.Cu at (408.9, 123.3)
Other:
- board text added: "but why on earth should that mean that it is not real?{dblquote}"
- board text added: "splinch"
- board text added: "v1 - made by Eyal Birger"
- board text added: "{dblquote}Of course it is happening inside your head, Harry,"
